Commit message: Drive: remove the DCC1000-era host PID, raise speed, acceleration and rate
The DCC1020 closes each wheel's speed loop on board, so the host wheel PIDs
and the limits chosen around the DCC1000 are no longer needed.

- isaacbot_amr_controller: delete SeededPidController / WheelSpeedLoop, their
  tests, plugin export and the launch file's chained-spawner logic. The
  package is now config, launch and Python tools only. wheel_step_response
  records joint_states (step reference turned into wheel speeds) instead of
  the PIDs' controller_state topics, which no longer exist.
- wheel_01_controller.yaml: controller_manager and diff_drive at 50 Hz (was
  25 Hz for the DCC1000's async-call latency); linear 1.2 m/s, angular
  1.5 rad/s (outer rim 1.968 m/s, ~5 % under the 12.58 rad/s DCC1020 clamp);
  acceleration 2.7 m/s^2 / 3.74 rad/s^2 (SWRS targets, ASSUMPTION until
  confirmed on the ground); jerk limit off (it smoothed 40 ms steps at 25 Hz).
- URDF: board ramp 6300 RPM/s, just above the worst wheel demand at the
  diff_drive limits, so diff_drive owns body acceleration; wheel joint limit
  12.58 rad/s (= the clamp); error debounce 4 cycles (80 ms at 50 Hz);
  velocity_command_zero_tolerance 0.01 (0.4 only covered the host PI's
  frozen integrator).
- ELRS teleop: caps 1.2 m/s / 1.5 rad/s, rim budget 1.97 m/s (the old 1.7
  kept headroom for the host PID's feed-forward), effective track 1.0236 m.
- Hardware interface: stale async/DCC1000 wording in comments only;
  encoderStaleTimeout renamed velocityStaleTimeout.
- Gazebo: sim_wheel_pid.yaml renamed sim_wheel_radius.yaml.
- SYS-SR-004 raised from 1.0 to 1.2 m/s in the SYS-SR xlsx (acceptance 1.26
  m/s; Revision History row added). MBSE parameters, architecture rates and
  compliance updated. SWRS .slreqx sets, model tests and exports still need a
  MATLAB build_all.
- Docs updated to match.

Co-Authored-By: Claude Opus 5.5 <noreply@anthropic.com>

File: isaacbot_amr_description/urdf/ardennes/ardennes_macro.urdf.xacro (robot description, xacro)
@@ -195,8 +195,9 @@
                message fields - never gates read()/write() return codes or triggers a lifecycle
                transition. The fault-flag category has no URDF param: it is hardcoded to 1
-               (immediate escalation, no debounce). -->
-          <param name="max_write_cmds_errors_count">2</param>
-          <param name="max_read_motor_states_errors_count">2</param>
-          <param name="max_read_driver_state_errors_count">2</param>
+               (immediate escalation, no debounce). Counted in controller_manager cycles: 4 at
+               50 Hz is the same 80 ms window that 2 was at 25 Hz. -->
+          <param name="max_write_cmds_errors_count">4</param>
+          <param name="max_read_motor_states_errors_count">4</param>
+          <param name="max_read_driver_state_errors_count">4</param>
           <!-- Max time (ms) since the last Phidget SDK telemetry callback (position/current/
                temperature) before a wheel driver is considered to have a communication error
@@ -222,6 +223,6 @@
                - wheels lifted or low speed, RC E-Stop in reach. -->
           <param name="motor_failsafe_enabled">true</param>
-          <!-- Brake (true) or coast (false) when the failsafe trips. Optional, default true - the
-               DCC1000 setup braked (braking strength 1.0); the DCC1020's own default is coast. -->
+          <!-- Brake (true) or coast (false) when the failsafe trips. Optional, default true, so a
+               tripped wheel stops instead of rolling on; the DCC1020's own default is coast. -->
           <param name="motor_failsafe_braking_enabled">true</param>
           <!-- DCC1020 motor current limit in A (checked against the board's range at configure).
@@ -267,12 +268,13 @@
           <!-- Zero-target band in which the controller lets go instead of holding the wheel. -->
           <param name="velocity_deadband_rpm">5</param>
-          <!-- On-board trapezoidal ramp, motor RPM/s. 1890 = 1.4 m/s^2 at the wheel
-               (1.4 / 0.1651 * 23.3 * 60 / 2pi), diff_drive's linear limit: the board interpolates
-               between diff_drive's 40 ms (25 Hz) command steps instead of jumping to each one.
-               Set on 2026-10-25 together with diff_drive's jerk limit (wheels lifted, see
-               wheel_01_controller.yaml). It caps each wheel on its own, so an accelerating turn
-               that asks the outer wheel for more than 1.4 m/s^2 (up to ~2.1 m/s^2 at the
-               diff_drive limits) is capped on that wheel - TBD: check turns on the ground. -->
-          <param name="motor_acceleration_rpm_s">1890</param>
+          <!-- On-board trapezoidal ramp, motor RPM/s. diff_drive owns the body acceleration
+               (wheel_01_controller.yaml); this only backs it up per wheel, and the board
+               interpolates between diff_drive's 20 ms (50 Hz) command steps. It sits just above
+               the worst wheel demand at the diff_drive limits, so it never caps an accelerating
+               turn: outer wheel 2.7 m/s^2 + 3.74 rad/s^2 * 0.5118 m = 4.61 m/s^2 = 27.9 rad/s^2
+               at r = 0.1651, * 23.3 * 60 / 2pi = 6213 RPM/s, rounded up. Was 1890 (= 1.4 m/s^2,
+               the DCC1000-era diff_drive limit). Whether the motors reach it at
+               motor_current_limit is TBD on the ground. -->
+          <param name="motor_acceleration_rpm_s">6300</param>
           <!-- Motor parameters -->
           <param name="motor_torque_constant">0.11</param>
@@ -294,14 +296,10 @@
                invariant (see domain/emergency_stop.cpp). Optional: omitting it keeps the
                compiled-in kDefaultVelocityCommandZeroTolerance (0.01).
-               Why 0.4 and not 0.01: with the DCC1000 the host wheel PIDs sat between diff_drive
-               and the hardware, and a frozen PI integrator kept a nonzero command (up to their
-               i_clamp_max) while motion was inhibited; 0.4 cleared that with a margin. Since the
-               DCC1020 swap there are no host PIDs - diff_drive's zero command reaches the
-               hardware as exactly 0 - so this can come back down toward 0.01 once that is
-               verified on the isaacbot.
-               This was previously 1.2 (~0.2 m/s at the A1's 0.1651 m wheel radius), which is
-               fast enough to walk beside and made the invariant largely decorative.
-               velocity_state_zero_tolerance below closes the real hazard regardless. -->
-          <param name="velocity_command_zero_tolerance">0.4</param>
+               0.01: diff_drive writes the wheel joints directly, so its zero command reaches the
+               hardware as exactly 0. It was 0.4 while host wheel PIDs sat in between (DCC1000
+               era): their frozen PI integrator kept a nonzero command while motion was
+               inhibited. velocity_state_zero_tolerance below closes the real hazard regardless.
+               TBD: confirm an E-Stop reset succeeds at rest on the isaacbot. -->
+          <param name="velocity_command_zero_tolerance">0.01</param>
           <!-- Deadband (rad/s at the wheel) below which a *measured* wheel velocity counts as
                "not moving", the second half of the same invariant. Unlike the command check

File: isaacbot_amr_description/urdf/common/wheel.urdf.xacro (robot description, xacro)
@@ -40,5 +40,7 @@
       <origin xyz="0.0 0.0 0.0" rpy="0.0 0.0 0.0" />
       <axis xyz="0.0 1.0 0.0" />
-      <limit effort="64.5" velocity="10.958" />
+      <!-- velocity: the DCC1020 target clamp, max_rpm_motor_speed 2800 * 2pi/60 / gear_ratio 23.3
+           = 12.58 rad/s at the wheel (ardennes_macro.urdf.xacro). -->
+      <limit effort="64.5" velocity="12.58" />
       <dynamics damping="0.01" friction="0.1" />
     </joint>
